Commit message: Add Mesh to URDF
Signed-off-by: Mickael Gaillard <mickael.gaillard@tactfactory.com>

File: picar_description/urdf/config.urdf.xacro (robot description, xacro)
@@ -3,10 +3,15 @@
   <xacro:arg name="body_mass"     default="1.000"/>
   <xacro:arg name="body_width"    default="0.078"/>
-  <xacro:arg name="body_length"   default="0.220"/>
-  <xacro:arg name="body_height"   default="0.030"/>
+  <xacro:arg name="body_length"   default="0.210"/>
+  <xacro:arg name="body_height"   default="0.029"/>
   <xacro:arg name="body_offset"   default="0.070"/>
   <xacro:arg name="wheelbase"     default="0.140"/>
-  <xacro:arg name="wheel_mass"    default="1.000"/>
-  <xacro:arg name="wheel_width"   default="0.030"/>
+  <!-- Rear wheel -->
+  <xacro:arg name="wheel_mass"    default="0.025"/>
+  <xacro:arg name="wheel_width"   default="0.0255"/>
+  <xacro:arg name="wheel_radius"  default="0.0335"/>
+  <!-- Rear wheel -->
+  <xacro:arg name="wheel_mass"    default="0.023"/>
+  <xacro:arg name="wheel_width"   default="0.026"/>
   <xacro:arg name="wheel_radius"  default="0.0335"/>
   <xacro:arg name="ground_clearance" default="0.2"/>

File: picar_description/urdf/picar.urdf.xacro (robot description, xacro)
@@ -12,14 +12,16 @@
   <link name="body">
     <visual>
-      <origin xyz="${body_offset} 0.0 0.0"/>
+      <origin xyz="0.0 0.0 ${-0.029/2}"/>
       <geometry>
-        <box size="${body_length} ${body_width} ${body_height}"/>
+        <!-- <box size="${body_length} ${body_width} ${body_height}" scale="0.001 0.001 0.001"/> -->
+        <mesh filename="package://picar_description/meshes/Chassis.dae"/>
       </geometry>
       <material name="body"/>
     </visual>
     <collision>
-      <origin xyz="${body_offset} 0.0 0.0"/>
+      <origin xyz="0.0 0.0 ${-0.029/2}"/>
       <geometry>
-        <box size="${body_length} ${body_width} ${body_height}"/>
+        <!-- <box size="${body_length} ${body_width} ${body_height}"/> -->
+        <mesh filename="package://picar_description/meshes/Chassis.dae"/>
       </geometry>
     </collision>
@@ -44,5 +46,5 @@
         <parent link="body"/>
         <child link="front_right_wheel_steering"/>
-        <origin rpy="0 0 ${pi}" xyz="${wheelbase} 0.04 0"/>
+        <origin rpy="0 0 ${pi}" xyz="${wheelbase} 0.048 0"/>
         <limit effort="5000" lower="-0.8" upper="0.8" velocity="1"/>
         <axis xyz="0 0 1"/>
@@ -66,11 +68,13 @@
         <visual>
           <geometry>
+            <!-- <cylinder length="${wheel_width}" radius="${wheel_radius}"/> -->
+            <mesh filename="package://picar_description/meshes/WheelFrontRight.dae"/>
+          </geometry>
+          <material name="rubber"/>
+        </visual>
+        <collision>
+          <geometry>
             <cylinder length="${wheel_width}" radius="${wheel_radius}"/>
-          </geometry>
-          <material name="rubber"/>
-        </visual>
-        <collision>
-          <geometry>
-            <cylinder length="${wheel_width}" radius="${wheel_radius}"/>
+            <mesh filename="package://picar_description/meshes/WheelFrontRight.dae"/>
           </geometry>
         </collision>
@@ -100,5 +104,5 @@
         <parent link="body"/>
         <child link="front_left_wheel_steering"/>
-        <origin rpy="0 0 ${pi}" xyz="${wheelbase} -0.04 0"/>
+        <origin rpy="0 0 ${pi}" xyz="${wheelbase} -0.048 0"/>
         <limit effort="5000" lower="-0.8" upper="0.8" velocity="1"/>
         <axis xyz="0 0 1"/>
@@ -122,11 +126,13 @@
         <visual>
           <geometry>
-            <cylinder length="${wheel_width}" radius="${wheel_radius}"/>
-          </geometry>
-          <material name="rubber"/>
-        </visual>
-        <collision>
-          <geometry>
-            <cylinder length="${wheel_width}" radius="${wheel_radius}"/>
+            <!-- <cylinder length="${wheel_width}" radius="${wheel_radius}"/> -->
+            <mesh filename="package://picar_description/meshes/WheelFrontLeft.dae"/>
+          </geometry>
+          <material name="rubber"/>
+        </visual>
+        <collision>
+          <geometry>
+            <!-- <cylinder length="${wheel_width}" radius="${wheel_radius}"/> -->
+            <mesh filename="package://picar_description/meshes/WheelFrontLeft.dae"/>
           </geometry>
         </collision>
@@ -166,11 +172,13 @@
         <visual>
           <geometry>
-            <cylinder length="${wheel_width}" radius="${wheel_radius}"/>
-          </geometry>
-          <material name="rubber"/>
-        </visual>
-        <collision>
-          <geometry>
-            <cylinder length="${wheel_width}" radius="${wheel_radius}"/>
+            <!-- <cylinder length="${wheel_width}" radius="${wheel_radius}"/> -->
+            <mesh filename="package://picar_description/meshes/WheelRearRight.dae"/>
+          </geometry>
+          <material name="rubber"/>
+        </visual>
+        <collision>
+          <geometry>
+            <!-- <cylinder length="${wheel_width}" radius="${wheel_radius}"/> -->
+            <mesh filename="package://picar_description/meshes/WheelRearRight.dae"/>
           </geometry>
         </collision>
@@ -208,11 +216,13 @@
         <visual>
           <geometry>
-            <cylinder length="${wheel_width}" radius="${wheel_radius}"/>
-          </geometry>
-          <material name="rubber"/>
-        </visual>
-        <collision>
-          <geometry>
-            <cylinder length="${wheel_width}" radius="${wheel_radius}"/>
+            <!-- <cylinder length="${wheel_width}" radius="${wheel_radius}"/> -->
+            <mesh filename="package://picar_description/meshes/WheelRearLeft.dae"/>
+          </geometry>
+          <material name="rubber"/>
+        </visual>
+        <collision>
+          <geometry>
+            <!-- <cylinder length="${wheel_width}" radius="${wheel_radius}"/> -->
+            <mesh filename="package://picar_description/meshes/WheelRearLeft.dae"/>
           </geometry>
         </collision>

Commit message: split front/rear wheel
Signed-off-by: Mickael Gaillard <mick.gaillard@gmail.com>

File: picar_description/urdf/config.urdf.xacro (robot description, xacro)
@@ -8,11 +8,11 @@
   <xacro:arg name="wheelbase"     default="0.140"/>
   <!-- Rear wheel -->
-  <xacro:arg name="wheel_mass"    default="0.025"/>
-  <xacro:arg name="wheel_width"   default="0.0255"/>
-  <xacro:arg name="wheel_radius"  default="0.0335"/>
+  <xacro:arg name="wheel_rear_mass"    default="0.025"/>
+  <xacro:arg name="wheel_rear_width"   default="0.0255"/>
+  <xacro:arg name="wheel_rear_radius"  default="0.0335"/>
   <!-- Rear wheel -->
-  <xacro:arg name="wheel_mass"    default="0.023"/>
-  <xacro:arg name="wheel_width"   default="0.026"/>
-  <xacro:arg name="wheel_radius"  default="0.0335"/>
+  <xacro:arg name="wheel_front_mass"    default="0.023"/>
+  <xacro:arg name="wheel_front_width"   default="0.026"/>
+  <xacro:arg name="wheel_front_radius"  default="0.0335"/>
   <xacro:arg name="ground_clearance" default="0.2"/>
   <xacro:include filename="$(find picar_description)/urdf/converter.urdf.xacro"/>

File: picar_description/urdf/converter.urdf.xacro (robot description, xacro)
@@ -7,7 +7,10 @@
   <xacro:property name="body_offset" value="$(arg body_offset)"/>
   <xacro:property name="wheelbase" value="$(arg wheelbase)"/>
-  <xacro:property name="wheel_mass" value="$(arg wheel_mass)"/>
-  <xacro:property name="wheel_width" value="$(arg wheel_width)"/>
-  <xacro:property name="wheel_radius" value="$(arg wheel_radius)"/>
+  <xacro:property name="wheel_rear_mass" value="$(arg wheel_rear_mass)"/>
+  <xacro:property name="wheel_rear_width" value="$(arg wheel_rear_width)"/>
+  <xacro:property name="wheel_rear_radius" value="$(arg wheel_rear_radius)"/>
+  <xacro:property name="wheel_front_mass" value="$(arg wheel_front_mass)"/>
+  <xacro:property name="wheel_front_width" value="$(arg wheel_front_width)"/>
+  <xacro:property name="wheel_front_radius" value="$(arg wheel_front_radius)"/>
   <xacro:property name="ground_clearance" value="$(arg ground_clearance)"/>
 </robot>

File: picar_description/urdf/picar.urdf.xacro (robot description, xacro)
@@ -6,22 +6,33 @@
     <plugin name="gazebo_ros_control" filename="libgazebo_ros_control.so">
       <robotNamespace>/picar</robotNamespace>
+      <!-- <robotSimType>steer_bot_hardware_gazebo/SteerBotHardwareGazebo</robotSimType> Not maintening -->
+      <!-- <robotSimType>gazebo_ros_control/DefaultRobotHWSim</robotSimType> -->
     </plugin>
   </gazebo>
+  <link name="world"/>
+  <joint name="fixed" type="fixed">
+    <parent link="world"/>
+    <child link="base_link"/>
+  </joint>
   <!-- Start Baselink -->
-  <link name="base_link"/>
+  <link name="base_link" >
+    <gazebo>
+      <material>Gazebo/Orange</material>
+    </gazebo>
+  </link>
   <link name="body">
     <visual>
-      <origin xyz="0.0 0.0 ${-0.029/2}"/>
+      <origin xyz="0.0 0.0 ${-body_height/2}"/>
+      <!-- ${body_offset} -->
       <geometry>
-        <!-- <box size="${body_length} ${body_width} ${body_height}" scale="0.001 0.001 0.001"/> -->
-        <mesh filename="package://picar_description/meshes/Chassis.dae"/>
+        <!-- <box size="${body_length} ${body_width} ${body_height}"/> -->
+        <mesh filename="package://picar_description/meshes/Chassis.dae" />
       </geometry>
       <material name="body"/>
     </visual>
     <collision>
-      <origin xyz="0.0 0.0 ${-0.029/2}"/>
+      <origin xyz="0.0 0.0 ${-body_height/2}"/>
       <geometry>
-        <!-- <box size="${body_length} ${body_width} ${body_height}"/> -->
-        <mesh filename="package://picar_description/meshes/Chassis.dae"/>
+        <mesh filename="package://picar_description/meshes/Chassis.dae" />
       </geometry>
     </collision>
@@ -58,5 +69,5 @@
       </link>
       <joint name="front_right_wheel_spinning_joint" type="continuous">
-        <origin rpy="${-pi/2} 0 0" xyz="0 ${-wheel_width/2} 0"/>
+        <origin rpy="${-pi/2} 0 0" xyz="0 ${-wheel_front_width/2} 0"/>
         <parent link="front_right_wheel_steering"/>
         <child link="front_right_wheel_spinning"/>
@@ -68,5 +79,5 @@
         <visual>
           <geometry>
-            <!-- <cylinder length="${wheel_width}" radius="${wheel_radius}"/> -->
+            <!-- <cylinder length="${wheel_front_width}" radius="${wheel_front_radius}"/> -->
             <mesh filename="package://picar_description/meshes/WheelFrontRight.dae"/>
           </geometry>
@@ -75,13 +86,13 @@
         <collision>
           <geometry>
-            <cylinder length="${wheel_width}" radius="${wheel_radius}"/>
+            <!-- <cylinder length="${wheel_front_width}" radius="${wheel_front_radius}"/> -->
             <mesh filename="package://picar_description/meshes/WheelFrontRight.dae"/>
           </geometry>
         </collision>
         <inertial>
-          <mass value="${wheel_mass}"/>
-          <inertia ixx="${wheel_mass*(3.0*wheel_radius*wheel_radius + wheel_width*wheel_width)/12.0}" ixy="0" ixz="0"
-                   iyy="${wheel_mass*(3.0*wheel_radius*wheel_radius + wheel_width*wheel_width)/12.0}" iyz="0"
-                   izz="${wheel_mass*wheel_radius*wheel_radius/2.0}"/>
+          <mass value="${wheel_front_mass}"/>
+          <inertia ixx="${wheel_front_mass*(3.0*wheel_front_radius*wheel_front_radius + wheel_front_width*wheel_front_width)/12.0}" ixy="0" ixz="0"
+                   iyy="${wheel_front_mass*(3.0*wheel_front_radius*wheel_front_radius + wheel_front_width*wheel_front_width)/12.0}" iyz="0"
+                   izz="${wheel_front_mass*wheel_front_radius*wheel_front_radius/2.0}"/>
         </inertial>
       </link>
@@ -116,5 +127,5 @@
       </link>
       <joint name="front_left_wheel_spinning_joint" type="continuous">
-        <origin rpy="${-pi/2} 0 0" xyz="0 ${wheel_width/2} 0"/>
+        <origin rpy="${-pi/2} 0 0" xyz="0 ${wheel_front_width/2} 0"/>
         <parent link="front_left_wheel_steering"/>
         <child link="front_left_wheel_spinning"/>
@@ -126,5 +137,5 @@
         <visual>
           <geometry>
-            <!-- <cylinder length="${wheel_width}" radius="${wheel_radius}"/> -->
+            <!-- <cylinder length="${wheel_front_width}" radius="${wheel_front_radius}"/> -->
             <mesh filename="package://picar_description/meshes/WheelFrontLeft.dae"/>
           </geometry>
@@ -133,13 +144,13 @@
         <collision>
           <geometry>
-            <!-- <cylinder length="${wheel_width}" radius="${wheel_radius}"/> -->
+            <!-- <cylinder length="${wheel_front_width}" radius="${wheel_front_radius}"/> -->
             <mesh filename="package://picar_description/meshes/WheelFrontLeft.dae"/>
           </geometry>
         </collision>
         <inertial>
-          <mass value="${wheel_mass}"/>
-          <inertia ixx="${wheel_mass*(3.0*wheel_radius*wheel_radius + wheel_width*wheel_width)/12.0}" ixy="0" ixz="0"
-                   iyy="${wheel_mass*(3.0*wheel_radius*wheel_radius + wheel_width*wheel_width)/12.0}" iyz="0"
-                   izz="${wheel_mass*wheel_radius*wheel_radius/2.0}"/>
+          <mass value="${wheel_front_mass}"/>
+          <inertia ixx="${wheel_front_mass*(3.0*wheel_front_radius*wheel_front_radius + wheel_front_width*wheel_front_width)/12.0}" ixy="0" ixz="0"
+                   iyy="${wheel_front_mass*(3.0*wheel_front_radius*wheel_front_radius + wheel_front_width*wheel_front_width)/12.0}" iyz="0"
+                   izz="${wheel_front_mass*wheel_front_radius*wheel_front_radius/2.0}"/>
         </inertial>
       </link>
@@ -172,5 +183,5 @@
         <visual>
           <geometry>
-            <!-- <cylinder length="${wheel_width}" radius="${wheel_radius}"/> -->
+            <!-- <cylinder length="${wheel_rear_width}" radius="${wheel_rear_radius}"/> -->
             <mesh filename="package://picar_description/meshes/WheelRearRight.dae"/>
           </geometry>
@@ -179,13 +190,13 @@
         <collision>
           <geometry>
-            <!-- <cylinder length="${wheel_width}" radius="${wheel_radius}"/> -->
+            <!-- <cylinder length="${wheel_rear_width}" radius="${wheel_rear_radius}"/> -->
             <mesh filename="package://picar_description/meshes/WheelRearRight.dae"/>
           </geometry>
         </collision>
         <inertial>
-          <mass value="${wheel_mass}"/>
-          <inertia ixx="${wheel_mass*(3.0*wheel_radius*wheel_radius + wheel_width*wheel_width)/12.0}" ixy="0" ixz="0"
-                   iyy="${wheel_mass*(3.0*wheel_radius*wheel_radius + wheel_width*wheel_width)/12.0}" iyz="0"
-                   izz="${wheel_mass*wheel_radius*wheel_radius/2.0}"/>
+          <mass value="${wheel_rear_mass}"/>
+          <inertia ixx="${wheel_rear_mass*(3.0*wheel_rear_radius*wheel_rear_radius + wheel_rear_width*wheel_rear_width)/12.0}" ixy="0" ixz="0"
+                   iyy="${wheel_rear_mass*(3.0*wheel_rear_radius*wheel_rear_radius + wheel_rear_width*wheel_rear_width)/12.0}" iyz="0"
+                   izz="${wheel_rear_mass*wheel_rear_radius*wheel_rear_radius/2.0}"/>
         </inertial>
       </link>
@@ -198,4 +209,5 @@
         </joint>
         <actuator name="rear_right_wheel_spinning_motor">
+          <hardwareInterface>VelocityJointInterface</hardwareInterface>
           <mechanicalReduction>1</mechanicalReduction>
         </actuator>
@@ -216,5 +228,5 @@
         <visual>
           <geometry>
-            <!-- <cylinder length="${wheel_width}" radius="${wheel_radius}"/> -->
+            <!-- <cylinder length="${wheel_rear_width}" radius="${wheel_rear_radius}"/> -->
             <mesh filename="package://picar_description/meshes/WheelRearLeft.dae"/>
           </geometry>
@@ -223,13 +235,13 @@
         <collision>
           <geometry>
-            <!-- <cylinder length="${wheel_width}" radius="${wheel_radius}"/> -->
+            <!-- <cylinder length="${wheel_rear_width}" radius="${wheel_rear_radius}"/> -->
             <mesh filename="package://picar_description/meshes/WheelRearLeft.dae"/>
           </geometry>
         </collision>
         <inertial>
-          <mass value="${wheel_mass}"/>
-          <inertia ixx="${wheel_mass*(3.0*wheel_radius*wheel_radius + wheel_width*wheel_width)/12.0}" ixy="0" ixz="0"
-                   iyy="${wheel_mass*(3.0*wheel_radius*wheel_radius + wheel_width*wheel_width)/12.0}" iyz="0"
-                   izz="${wheel_mass*wheel_radius*wheel_radius/2.0}"/>
+          <mass value="${wheel_rear_mass}"/>
+          <inertia ixx="${wheel_rear_mass*(3.0*wheel_rear_radius*wheel_rear_radius + wheel_rear_width*wheel_rear_width)/12.0}" ixy="0" ixz="0"
+                   iyy="${wheel_rear_mass*(3.0*wheel_rear_radius*wheel_rear_radius + wheel_rear_width*wheel_rear_width)/12.0}" iyz="0"
+                   izz="${wheel_rear_mass*wheel_rear_radius*wheel_rear_radius/2.0}"/>
         </inertial>
       </link>
@@ -242,4 +254,5 @@
         </joint>
         <actuator name="rear_left_wheel_spinning_motor">
+          <hardwareInterface>VelocityJointInterface</hardwareInterface>
           <mechanicalReduction>1</mechanicalReduction>
         </actuator>
