Commit message: push gazebo support
Signed-off-by: Mickael Gaillard <mick.gaillard@gmail.com>

File: picar_description/urdf/converter.urdf.xacro (robot description, xacro)
@@ -10,4 +10,5 @@
   <xacro:property name="wheel_rear_width" value="$(arg wheel_rear_width)"/>
   <xacro:property name="wheel_rear_radius" value="$(arg wheel_rear_radius)"/>
+  <xacro:property name="steer_front_mass" value="$(arg steer_front_mass)"/>
   <xacro:property name="wheel_front_mass" value="$(arg wheel_front_mass)"/>
   <xacro:property name="wheel_front_width" value="$(arg wheel_front_width)"/>

File: picar_description/urdf/picar.urdf.xacro (robot description, xacro)
@@ -1,12 +1,20 @@
-<?xml version="1.0"?>
+<?xml version="1.0" ?>
+<!--
+  Robot model adapted from :
+  - https://github.com/CIR-KIT/steer_drive_ros/blob/kinetic-devel/steer_drive_controller/test/common/urdf/steerbot.xacro
+  - https://github.com/srmainwaring/steer_bot/blob/master/steer_bot_description/urdf/steer_bot.urdf.xacro
+-->
 <robot name="picar" xmlns:xacro="http://www.ros.org/wiki/xacro">
   <xacro:include filename="$(find picar_description)/urdf/config.xacro" />
   <xacro:include filename="$(find picar_description)/urdf/materials.xacro" />
   <xacro:include filename="$(find picar_description)/urdf/inertials.xacro" />
+  <xacro:property name="robot_namespace" value="/picar"/>
+  <!-- Gazebo plugins -->
   <gazebo>
-    <plugin name="gazebo_ros_control" filename="libgazebo_ros_control.so">
-      <robotNamespace>/picar</robotNamespace>
+    <!-- Load ros_control plugin using the steer_bot_hardware_gazebo
+    implementation of the hardware_interface::RobotHW -->
+    <plugin filename="libgazebo_ros_control.so" name="gazebo_ros_control">
+      <robotNamespace>${robot_namespace}</robotNamespace>
       <robotSimType>steer_bot_hardware_gazebo/SteerBotHardwareGazebo</robotSimType>
-      <robotSimType>picar_hardware_gazebo/PicarHardwareGazebo</robotSimType>
       <legacyModeNS>false</legacyModeNS>
     </plugin>
@@ -28,41 +36,127 @@
     <xacro:solid_cuboid_inertial xyz="0.0 0.0 ${body_height/2}" rpy="0.0 0.0 0.0" mass="${body_mass}" x="${body_length}" y="${body_width}" z="${body_height}" />
   </link>
+  <gazebo reference="base_link">
+    <material>Gazebo/Green</material>
+  </gazebo>
   <!-- End Baselink -->
+  <link name="front_steer_link">
+    <!--visual>
+      <origin rpy="0 0 0" xyz="0 0 0"/>
+      <geometry>
+        <cylinder length="0.002" radius="0.005"/>
+      </geometry>
+      <material name="yellow"/>
+    </visual-->
+    <!--collision>
+      <origin rpy="0 0 0" xyz="0 0 0"/>
+      <geometry>
+        <cylinder length="0.02" radius="0.05"/>
+      </geometry>
+    </collision-->
+    <inertial>
+      <origin rpy="0 0 0" xyz="0 0 0"/>
+      <mass value="0.03125"/>
+      <inertia ixx="0.0006583333333333334" ixy="0.0" ixz="0.0" iyy="0.0006583333333333334" iyz="0.0" izz="0.0012500000000000002"/>
+    </inertial>
+  </link>
+  <joint name="front_steer_joint" type="revolute">
+    <parent link="base_link"/>
+    <child link="front_steer_link"/>
+    <origin rpy="0 0 0" xyz="0.2 0 0.12000000000000001"/>
+    <axis xyz="0 0 1"/>
+    <limit effort="10.0" lower="${-pi}" upper="${pi}" velocity="5.0"/>
+    <dynamics damping="0.7" friction="0.1" />
+  </joint>
+  <transmission name="front_steer_joint_trans">
+    <type>transmission_interface/SimpleTransmission</type>
+    <actuator name="front_steer_joint_motor">
+      <mechanicalReduction>1</mechanicalReduction>
+      <hardwareInterface>hardware_interface/PositionJointInterface</hardwareInterface>
+    </actuator>
+    <joint name="front_steer_joint">
+      <hardwareInterface>hardware_interface/PositionJointInterface</hardwareInterface>
+    </joint>
+  </transmission>
+  <gazebo reference="front_steer_link">
+    <material>Gazebo/Yellow</material>
+  </gazebo>
+  <link name="rear_wheel_link">
+    <visual>
+      <origin rpy="0 0 0" xyz="0 0 0"/>
+      <geometry>
+        <cylinder length="0.08" radius="0.005"/>
+      </geometry>
+      <material name="yellow"/>
+    </visual>
+    <!--collision>
+      <origin rpy="0 0 0" xyz="0 0 0"/>
+      <geometry>
+        <cylinder length="0.04" radius="0.025"/>
+      </geometry>
+    </collision-->
+    <inertial>
+      <origin rpy="0 0 0" xyz="0 0 0"/>
+      <mass value="0.03125"/>
+      <inertia ixx="9.049479166666668e-06" ixy="0.0" ixz="0.0" iyy="9.049479166666668e-06" iyz="0.0" izz="9.765625000000002e-06"/>
+    </inertial>
+  </link>
+  <joint name="rear_wheel_joint" type="continuous">
+    <parent link="base_link"/>
+    <child link="rear_wheel_link"/>
+    <origin rpy="${-pi/2} 0 0" xyz="0 0 0"/>
+    <axis xyz="0 0 1"/>
+  </joint>
+  <transmission name="rear_wheel_joint_trans">
+    <type>transmission_interface/SimpleTransmission</type>
+    <actuator name="rear_wheel_joint_motor">
+      <mechanicalReduction>1</mechanicalReduction>
+      <hardwareInterface>hardware_interface/VelocityJointInterface</hardwareInterface>
+    </actuator>
+    <joint name="rear_wheel_joint">
+      <hardwareInterface>hardware_interface/VelocityJointInterface</hardwareInterface>
+    </joint>
+  </transmission>
+  <gazebo reference="rear_wheel_link">
+    <material>Gazebo/Yellow</material>
+  </gazebo>
   <!-- Start Front -->
   <!-- Start Front right -->
-  <!-- Start Join -->
-  <joint name="front_right_wheel_steering_joint" type="revolute">
-    <parent link="base_link" />
-    <child link="front_right_wheel_steering_link" />
-    <origin rpy="0.0 0.0 ${pi}" xyz="${wheelbase} 0.048 0.0" />
-    <limit effort="5000" lower="-0.8" upper="0.8" velocity="1" />
-    <axis xyz="0 0 1" />
-    <dynamics damping="0.7" friction="0.1" />
-  </joint>
-  <joint name="front_right_wheel_spinning_joint" type="continuous">
-    <origin rpy="${-pi/2} 0.0 0.0" xyz="0.0 ${-wheel_front_width/2} 0.0" />
-    <parent link="front_right_wheel_steering_link" />
-    <child link="front_right_wheel_spinning_link" />
-    <axis xyz="0 0 -1" />
-  </joint>
-  <!-- End Join -->
-  <!-- Start Visual -->
-  <link name="front_right_wheel_steering_link">
-    <inertial>
-      <origin rpy="0.0 0.0 0.0" xyz="0.0 0.0 0.0" />
-      <mass value="0.1" />
-      <inertia ixx="5.6112500000000015e-05" ixy="0" ixz="0" iyy="5.6112500000000015e-05" iyz="0" izz="5.6112500000000015e-05" />
-    </inertial>
-  </link>
-  <link name="front_right_wheel_spinning_link">
-    <visual>
-      <origin rpy="0.0 0.0 0.0" xyz="0.0 0.0 0.0" />
+  <link name="front_right_steer_link">
+    <!--visual>
+      <origin rpy="0 0 0" xyz="0 0 0"/>
+      <geometry>
+        <cylinder length="0.02" radius="0.05"/>
+      </geometry>
+      <material name="blue"/>
+    </visual>
+    <collision>
+      <origin rpy="0 0 0" xyz="0 0 0"/>
+      <geometry>
+        <cylinder length="0.02" radius="0.05"/>
+      </geometry>
+    </collision-->
+    <inertial>
+      <origin rpy="0 0 0" xyz="0 0 0"/>
+      <mass value="${steer_front_mass}"/>
+      <inertia ixx="0.0006583333333333334" ixy="0.0" ixz="0.0" iyy="0.0006583333333333334" iyz="0.0" izz="0.0012500000000000002"/>
+    </inertial>
+  </link>
+  <joint name="front_right_steer_joint" type="revolute">
+    <parent link="base_link"/>
+    <child link="front_right_steer_link"/>
+    <origin rpy="0.0 0.0 ${pi}" xyz="${wheelbase} 0.048 0.0"/>
+    <axis xyz="0 -0 1"/>
+    <limit effort="10.0" lower="-0.7853981633974483" upper="0.7853981633974483" velocity="5.0"/>
+  </joint>
+  <link name="front_right_wheel_link">
+    <visual>
+      <origin rpy="0 0 0" xyz="0 0 0"/>
       <geometry>
         <mesh filename="package://picar_description/meshes/WheelFrontRight.dae" />
       </geometry>
-      <material name="rubber" />
-    </visual>
-    <collision>
-      <origin rpy="0.0 0.0 0.0" xyz="0.0 0.0 0.0" />
+      <material name="red"/>
+    </visual>
+    <collision>
+      <origin rpy="0 0 0" xyz="0 0 0"/>
       <geometry>
         <mesh filename="package://picar_description/meshes/WheelFrontRight.dae" />
@@ -70,68 +164,80 @@
     </collision>
     <inertial>
-      <origin rpy="0.0 0.0 0.0" xyz="0.0 0.0 0.0" />
-      <mass value="${wheel_front_mass}" />
-      <inertia ixx="${wheel_front_mass*(3.0*wheel_front_radius*wheel_front_radius + wheel_front_width*wheel_front_width)/12.0}" ixy="0" ixz="0" iyy="${wheel_front_mass*(3.0*wheel_front_radius*wheel_front_radius + wheel_front_width*wheel_front_width)/12.0}" iyz="0" izz="${wheel_front_mass*wheel_front_radius*wheel_front_radius/2.0}" />
-    </inertial>
-  </link>
-  <!-- End Visual -->
-  <!-- Start Transmission -->
-  <transmission name="front_right_wheel_steering_trans">
-    <type>transmission_interface/SimpleTransmission</type>
-    <actuator name="front_right_wheel_steering_motor">
-      <mechanicalReduction>1</mechanicalReduction>
-      <hardwareInterface>hardware_interface/PositionJointInterface</hardwareInterface>
-    </actuator>
-    <joint name="front_right_wheel_steering_joint">
-      <hardwareInterface>hardware_interface/PositionJointInterface</hardwareInterface>
-    </joint>
-  </transmission>
-  <transmission name="front_right_wheel_spinning_trans">
-    <type>transmission_interface/SimpleTransmission</type>
-    <actuator name="front_left_wheel_spinning_motor">
-      <mechanicalReduction>1</mechanicalReduction>
-      <hardwareInterface>hardware_interface/VelocityJointInterface</hardwareInterface>
-    </actuator>
-    <joint name="front_right_wheel_spinning_joint">
-      <hardwareInterface>hardware_interface/VelocityJointInterface</hardwareInterface>
-    </joint>
-  </transmission>
-  <!-- End Transmission -->
+      <origin rpy="0 0 0" xyz="0 0 0"/>
+      <mass value="${wheel_front_mass}"/>
+      <inertia ixx="${wheel_front_mass*(3.0*wheel_front_radius*wheel_front_radius + wheel_front_width*wheel_front_width)/12.0}" ixy="0" ixz="0" iyy="${wheel_front_mass*(3.0*wheel_front_radius*wheel_front_radius + wheel_front_width*wheel_front_width)/12.0}" iyz="0" izz="${wheel_front_mass*wheel_front_radius*wheel_front_radius/2.0}"/>
+    </inertial>
+  </link>
+  <joint name="front_right_wheel_joint" type="continuous">
+    <parent link="front_right_steer_link"/>
+    <child link="front_right_wheel_link"/>
+    <origin rpy="${-pi/2} 0.0 0.0" xyz="0.0 ${-wheel_front_width/2} 0.0"/>
+    <axis xyz="0 0 1"/>
+  </joint>
+  <transmission name="front_right_steer_joint_trans">
+    <type>transmission_interface/SimpleTransmission</type>
+    <actuator name="front_right_steer_joint_motor">
+      <mechanicalReduction>1</mechanicalReduction>
+      <hardwareInterface>hardware_interface/PositionJointInterface</hardwareInterface>
+    </actuator>
+    <joint name="front_right_steer_joint">
+      <hardwareInterface>hardware_interface/PositionJointInterface</hardwareInterface>
+    </joint>
+  </transmission>
+  <transmission name="front_right_wheel_joint_trans">
+    <type>transmission_interface/SimpleTransmission</type>
+    <actuator name="front_right_wheel_joint_motor">
+      <mechanicalReduction>1</mechanicalReduction>
+      <hardwareInterface>hardware_interface/VelocityJointInterface</hardwareInterface>
+    </actuator>
+    <joint name="front_right_wheel_joint">
+      <hardwareInterface>hardware_interface/VelocityJointInterface</hardwareInterface>
+    </joint>
+  </transmission>
+  <gazebo reference="front_right_steer_link">
+    <material>Gazebo/Blue</material>
+  </gazebo>
+  <gazebo reference="front_right_wheel_link">
+    <material>Gazebo/Red</material>
+  </gazebo>
   <!-- End Front right -->
   <!-- Start Front left -->
-  <!-- Start Join -->
-  <joint name="front_left_wheel_steering_joint" type="revolute">
-    <parent link="base_link" />
-    <child link="front_left_wheel_steering_link" />
-    <origin rpy="0 0 ${pi}" xyz="${wheelbase} -0.048 0" />
-    <limit effort="5000" lower="-0.8" upper="0.8" velocity="1" />
-    <axis xyz="0 0 1" />
-    <dynamics damping="0.7" friction="0.1" />
-  </joint>
-  <joint name="front_left_wheel_spinning_joint" type="continuous">
-    <origin rpy="${-pi/2} 0 0" xyz="0 ${wheel_front_width/2} 0" />
-    <parent link="front_left_wheel_steering_link" />
-    <child link="front_left_wheel_spinning_link" />
-    <axis xyz="0 0 -1" />
-  </joint>
-  <!-- End Join -->
-  <!-- Start Visual -->
-  <link name="front_left_wheel_steering_link">
-    <inertial>
-      <origin rpy="0.0 0.0 0.0" xyz="0.0 0.0 0.0" />
-      <mass value="0.1" />
-      <inertia ixx="5.6112500000000015e-05" ixy="0" ixz="0" iyy="5.6112500000000015e-05" iyz="0" izz="5.6112500000000015e-05" />
-    </inertial>
-  </link>
-  <link name="front_left_wheel_spinning_link">
-    <visual>
-      <origin rpy="0.0 0.0 0.0" xyz="0.0 0.0 0.0" />
+  <link name="front_left_steer_link">
+    <!--visual>
+      <origin rpy="0 0 0" xyz="0 0 0"/>
+      <geometry>
+        <cylinder length="0.02" radius="0.05"/>
+      </geometry>
+      <material name="blue"/>
+    </visual>
+    <collision>
+      <origin rpy="0 0 0" xyz="0 0 0"/>
+      <geometry>
+        <cylinder length="0.02" radius="0.05"/>
+      </geometry>
+    </collision-->
+    <inertial>
+      <origin rpy="0 0 0" xyz="0 0 0"/>
+      <mass value="${steer_front_mass}"/>
+      <inertia ixx="0.0006583333333333334" ixy="0.0" ixz="0.0" iyy="0.0006583333333333334" iyz="0.0" izz="0.0012500000000000002"/>
+    </inertial>
+  </link>
+  <joint name="front_left_steer_joint" type="revolute">
+    <parent link="base_link"/>
+    <child link="front_left_steer_link"/>
+    <origin rpy="0 0 ${pi}" xyz="${wheelbase} -0.048 0"/>
+    <axis xyz="0 0 1"/>
+    <limit effort="10.0" lower="-0.7853981633974483" upper="0.7853981633974483" velocity="5.0"/>
+  </joint>
+  <link name="front_left_wheel_link">
+    <visual>
+      <origin rpy="0 0 0" xyz="0 0 0"/>
       <geometry>
         <mesh filename="package://picar_description/meshes/WheelFrontLeft.dae" />
       </geometry>
-      <material name="rubber" />
-    </visual>
-    <collision>
-      <origin rpy="0.0 0.0 0.0" xyz="0.0 0.0 0.0" />
+      <material name="red"/>
+    </visual>
+    <collision>
+      <origin rpy="0 0 0" xyz="0 0 0"/>
       <geometry>
         <mesh filename="package://picar_description/meshes/WheelFrontLeft.dae" />
@@ -139,55 +245,55 @@
     </collision>
     <inertial>
-      <origin rpy="0.0 0.0 0.0" xyz="0.0 0.0 0.0" />
-      <mass value="${wheel_front_mass}" />
-      <inertia ixx="${wheel_front_mass*(3.0*wheel_front_radius*wheel_front_radius + wheel_front_width*wheel_front_width)/12.0}" ixy="0" ixz="0" iyy="${wheel_front_mass*(3.0*wheel_front_radius*wheel_front_radius + wheel_front_width*wheel_front_width)/12.0}" iyz="0" izz="${wheel_front_mass*wheel_front_radius*wheel_front_radius/2.0}" />
-    </inertial>
-  </link>
-  <!-- End Visual -->
-  <!-- Start Transmission -->
-  <transmission name="front_left_wheel_steering_trans">
-    <type>transmission_interface/SimpleTransmission</type>
-    <actuator name="front_left_wheel_steering_motor">
-      <mechanicalReduction>1</mechanicalReduction>
-      <hardwareInterface>hardware_interface/PositionJointInterface</hardwareInterface>
-    </actuator>
-    <joint name="front_left_wheel_steering_joint">
-      <hardwareInterface>hardware_interface/PositionJointInterface</hardwareInterface>
-    </joint>
-  </transmission>
-  <transmission name="front_left_wheel_spinning_trans">
-    <type>transmission_interface/SimpleTransmission</type>
-    <actuator name="front_left_wheel_spinning_motor">
-      <mechanicalReduction>1</mechanicalReduction>
-      <hardwareInterface>hardware_interface/VelocityJointInterface</hardwareInterface>
-    </actuator>
-    <joint name="front_left_wheel_spinning_joint">
-      <hardwareInterface>hardware_interface/VelocityJointInterface</hardwareInterface>
-    </joint>
-  </transmission>
-  <!-- End Transmission -->
+      <origin rpy="0 0 0" xyz="0 0 0"/>
+      <mass value="${wheel_front_mass}"/>
+      <inertia ixx="${wheel_front_mass*(3.0*wheel_front_radius*wheel_front_radius + wheel_front_width*wheel_front_width)/12.0}" ixy="0" ixz="0" iyy="${wheel_front_mass*(3.0*wheel_front_radius*wheel_front_radius + wheel_front_width*wheel_front_width)/12.0}" iyz="0" izz="${wheel_front_mass*wheel_front_radius*wheel_front_radius/2.0}"/>
+    </inertial>
+  </link>
+  <joint name="front_left_wheel_joint" type="continuous">
+    <parent link="front_left_steer_link"/>
+    <child link="front_left_wheel_link"/>
+    <origin rpy="${-pi/2} 0 0" xyz="0 ${wheel_front_width/2} 0"/>
+    <axis xyz="0 0 -1"/>
+  </joint>
+  <transmission name="front_left_steer_joint_trans">
+    <type>transmission_interface/SimpleTransmission</type>
+    <actuator name="front_left_steer_joint_motor">
+      <mechanicalReduction>1</mechanicalReduction>
+      <hardwareInterface>hardware_interface/PositionJointInterface</hardwareInterface>
+    </actuator>
+    <joint name="front_left_steer_joint">
+      <hardwareInterface>hardware_interface/PositionJointInterface</hardwareInterface>
+    </joint>
+  </transmission>
+  <transmission name="front_left_wheel_joint_trans">
+    <type>transmission_interface/SimpleTransmission</type>
+    <actuator name="front_left_wheel_joint_motor">
+      <mechanicalReduction>1</mechanicalReduction>
+      <hardwareInterface>hardware_interface/VelocityJointInterface</hardwareInterface>
+    </actuator>
+    <joint name="front_left_wheel_joint">
+      <hardwareInterface>hardware_interface/VelocityJointInterface</hardwareInterface>
+    </joint>
+  </transmission>
+  <gazebo reference="front_left_steer_link">
+    <material>Gazebo/Blue</material>
+  </gazebo>
+  <gazebo reference="front_left_wheel_link">
+    <material>Gazebo/Red</material>
+  </gazebo>
   <!-- End Front left -->
   <!-- End Front -->
   <!-- Start Rear -->
   <!-- Start Rear right -->
-  <!-- Start Join -->
-  <joint name="rear_right_wheel_spinning_joint" type="continuous">
-    <parent link="base_link" />
-    <child link="rear_right_wheel_spinning_link" />
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