Commit message: Fix Gazebo link
Signed-off-by: Mickael Gaillard <mick.gaillard@gmail.com>

File: picar_description/urdf/config.xacro (robot description, xacro)
@@ -8,9 +8,11 @@
   <xacro:arg name="wheelbase"     default="0.140"/>
   <!-- Rear wheel -->
+  <xacro:arg name="steer_rear_axe"     default="0.055"/>
   <xacro:arg name="wheel_rear_mass"    default="0.025"/>
   <xacro:arg name="wheel_rear_width"   default="0.0255"/>
   <xacro:arg name="wheel_rear_radius"  default="0.0335"/>
   <!-- Front wheel -->
-  <xacro:arg name="steer_front_mass"    default="0.001"/>
+  <xacro:arg name="steer_front_mass"    default="0.031"/>
+  <xacro:arg name="steer_front_axe"     default="0.048"/>
   <xacro:arg name="wheel_front_mass"    default="0.023"/>
   <xacro:arg name="wheel_front_width"   default="0.026"/>

File: picar_description/urdf/converter.urdf.xacro (robot description, xacro)
@@ -7,8 +7,10 @@
   <xacro:property name="body_offset" value="$(arg body_offset)"/>
   <xacro:property name="wheelbase" value="$(arg wheelbase)"/>
+  <xacro:property name="steer_rear_axe" value="$(arg steer_rear_axe)"/>
   <xacro:property name="wheel_rear_mass" value="$(arg wheel_rear_mass)"/>
   <xacro:property name="wheel_rear_width" value="$(arg wheel_rear_width)"/>
   <xacro:property name="wheel_rear_radius" value="$(arg wheel_rear_radius)"/>
   <xacro:property name="steer_front_mass" value="$(arg steer_front_mass)"/>
+  <xacro:property name="steer_front_axe"  value="$(arg steer_front_axe)"/>
   <xacro:property name="wheel_front_mass" value="$(arg wheel_front_mass)"/>
   <xacro:property name="wheel_front_width" value="$(arg wheel_front_width)"/>

File: picar_description/urdf/inertials.xacro (robot description, xacro)
@@ -21,8 +21,4 @@
                 izz="${mass * (x * x + y * y) / 12.0}">
             </inertia>
-            <!-- <inertia
-                ixx="${body_mass / 12.0 * (body_height*body_height + body_length*body_length)}" ixy="0.0" ixz="0.0"
-                iyy="${body_mass / 12.0 * (body_width*body_width + body_length*body_length)}" iyz="0.0"
-                izz="${body_mass / 12.0 * (body_width*body_width + body_height*body_height)}"/> -->
         </inertial>
     </xacro:macro>
@@ -42,5 +38,5 @@
         <inertial>
             <mass value="0.001"/>
-            <inertia ixx="0.001" ixy="0" ixz="0" iyy="0.001" iyz="0" izz="0.001"/>
+            <inertia ixx="9.049479166666668e-06" ixy="0" ixz="0" iyy="9.049479166666668e-06" iyz="0" izz="9.765625000000002e-06"/>
         </inertial>
     </xacro:macro>

File: picar_description/urdf/picar.urdf.xacro (robot description, xacro)
@@ -34,5 +34,11 @@
       </geometry>
     </collision>
-    <xacro:solid_cuboid_inertial xyz="0.0 0.0 ${body_height/2}" rpy="0.0 0.0 0.0" mass="${body_mass}" x="${body_length}" y="${body_width}" z="${body_height}" />
+    <xacro:solid_cuboid_inertial
+        xyz="0.0 0.0 ${body_height/2}"
+        rpy="0.0 0.0 0.0"
+        mass="${body_mass}"
+        x="${body_length}"
+        y="${body_width}"
+        z="${body_height}" />
   </link>
   <gazebo reference="base_link">
@@ -41,27 +47,16 @@
   <!-- End Baselink -->
   <link name="front_steer_link">
-    <!--visual>
-      <origin rpy="0 0 0" xyz="0 0 0"/>
-      <geometry>
-        <cylinder length="0.002" radius="0.005"/>
-      </geometry>
-      <material name="yellow"/>
-    </visual-->
-    <!--collision>
-      <origin rpy="0 0 0" xyz="0 0 0"/>
-      <geometry>
-        <cylinder length="0.02" radius="0.05"/>
-      </geometry>
-    </collision-->
-    <inertial>
-      <origin rpy="0 0 0" xyz="0 0 0"/>
-      <mass value="0.03125"/>
-      <inertia ixx="0.0006583333333333334" ixy="0.0" ixz="0.0" iyy="0.0006583333333333334" iyz="0.0" izz="0.0012500000000000002"/>
-    </inertial>
+    <xacro:solid_cylinder_inertial
+      xyz="0.0 0.0 0.0"
+      rpy="0.0 0.0 0.0"
+      mass="0.03125"
+      radius="0.01"
+      length="0.01"/>
+    <!--inertia ixx="0.0006583333333333334" ixy="0.0" ixz="0.0" iyy="0.0006583333333333334" iyz="0.0" izz="0.0012500000000000002"/-->
   </link>
   <joint name="front_steer_joint" type="revolute">
     <parent link="base_link"/>
     <child link="front_steer_link"/>
-    <origin rpy="0 0 0" xyz="0.2 0 0.12000000000000001"/>
+    <origin rpy="0.0 0.0 0.0" xyz="0.2 0 0.12000000000000001"/>
     <axis xyz="0 0 1"/>
     <limit effort="10.0" lower="${-pi}" upper="${pi}" velocity="5.0"/>
@@ -83,5 +78,5 @@
   <link name="rear_wheel_link">
     <visual>
-      <origin rpy="0 0 0" xyz="0 0 0"/>
+      <origin rpy="0.0 0.0 0.0" xyz="0.0 0.0 0.0"/>
       <geometry>
         <cylinder length="0.08" radius="0.005"/>
@@ -89,20 +84,13 @@
       <material name="yellow"/>
     </visual>
-    <!--collision>
-      <origin rpy="0 0 0" xyz="0 0 0"/>
-      <geometry>
-        <cylinder length="0.04" radius="0.025"/>
-      </geometry>
-    </collision-->
-    <inertial>
-      <origin rpy="0 0 0" xyz="0 0 0"/>
+    <xacro:null_inertial />
+    <!--inertial>
       <mass value="0.03125"/>
-      <inertia ixx="9.049479166666668e-06" ixy="0.0" ixz="0.0" iyy="9.049479166666668e-06" iyz="0.0" izz="9.765625000000002e-06"/>
-    </inertial>
+    </inertial-->
   </link>
   <joint name="rear_wheel_joint" type="continuous">
     <parent link="base_link"/>
     <child link="rear_wheel_link"/>
-    <origin rpy="${-pi/2} 0 0" xyz="0 0 0"/>
+    <origin rpy="${-pi/2} 0.0 0.0" xyz="0.0 0.0 0.0"/>
     <axis xyz="0 0 1"/>
   </joint>
@@ -123,54 +111,46 @@
   <!-- Start Front right -->
   <link name="front_right_steer_link">
-    <!--visual>
-      <origin rpy="0 0 0" xyz="0 0 0"/>
-      <geometry>
-        <cylinder length="0.02" radius="0.05"/>
-      </geometry>
-      <material name="blue"/>
-    </visual>
-    <collision>
-      <origin rpy="0 0 0" xyz="0 0 0"/>
-      <geometry>
-        <cylinder length="0.02" radius="0.05"/>
-      </geometry>
-    </collision-->
-    <inertial>
-      <origin rpy="0 0 0" xyz="0 0 0"/>
-      <mass value="${steer_front_mass}"/>
+    <xacro:solid_cylinder_inertial
+      xyz="0.0 0.0 0.0"
+      rpy="0.0 0.0 0.0"
+      mass="${steer_front_mass}"
+      radius="0.01"
+      length="0.01"/>
+    <!--inertial>
       <inertia ixx="0.0006583333333333334" ixy="0.0" ixz="0.0" iyy="0.0006583333333333334" iyz="0.0" izz="0.0012500000000000002"/>
-    </inertial>
+    </inertial-->
   </link>
   <joint name="front_right_steer_joint" type="revolute">
     <parent link="base_link"/>
     <child link="front_right_steer_link"/>
-    <origin rpy="0.0 0.0 ${pi}" xyz="${wheelbase} 0.048 0.0"/>
-    <axis xyz="0 -0 1"/>
+    <origin rpy="0.0 0.0 0.0" xyz="${wheelbase} ${steer_front_axe} 0.0"/>
+    <axis xyz="0 0 1"/>
     <limit effort="10.0" lower="-0.7853981633974483" upper="0.7853981633974483" velocity="5.0"/>
   </joint>
   <link name="front_right_wheel_link">
     <visual>
-      <origin rpy="0 0 0" xyz="0 0 0"/>
+      <origin rpy="0.0 0.0 0.0" xyz="0.0 0.0 0.0"/>
       <geometry>
         <mesh filename="package://picar_description/meshes/WheelFrontRight.dae" />
       </geometry>
-      <material name="red"/>
-    </visual>
-    <collision>
-      <origin rpy="0 0 0" xyz="0 0 0"/>
+      <!--material name="red"/-->
+    </visual>
+    <collision>
+      <origin rpy="0.0 0.0 0.0" xyz="0.0 0.0 0.0"/>
       <geometry>
         <mesh filename="package://picar_description/meshes/WheelFrontRight.dae" />
       </geometry>
     </collision>
-    <inertial>
-      <origin rpy="0 0 0" xyz="0 0 0"/>
-      <mass value="${wheel_front_mass}"/>
-      <inertia ixx="${wheel_front_mass*(3.0*wheel_front_radius*wheel_front_radius + wheel_front_width*wheel_front_width)/12.0}" ixy="0" ixz="0" iyy="${wheel_front_mass*(3.0*wheel_front_radius*wheel_front_radius + wheel_front_width*wheel_front_width)/12.0}" iyz="0" izz="${wheel_front_mass*wheel_front_radius*wheel_front_radius/2.0}"/>
-    </inertial>
+    <xacro:solid_cylinder_inertial
+      xyz="0.0 0.0 0.0"
+      rpy="0.0 0.0 0.0"
+      mass="${wheel_front_mass}"
+      radius="${wheel_front_radius}"
+      length="${wheel_front_width}"/>
   </link>
   <joint name="front_right_wheel_joint" type="continuous">
     <parent link="front_right_steer_link"/>
     <child link="front_right_wheel_link"/>
-    <origin rpy="${-pi/2} 0.0 0.0" xyz="0.0 ${-wheel_front_width/2} 0.0"/>
+    <origin rpy="${-pi/2} 0.0 0.0" xyz="0.0 ${-wheel_front_width/2+wheel_front_width} 0.0"/>
     <axis xyz="0 0 1"/>
   </joint>
@@ -204,27 +184,18 @@
   <!-- Start Front left -->
   <link name="front_left_steer_link">
-    <!--visual>
-      <origin rpy="0 0 0" xyz="0 0 0"/>
-      <geometry>
-        <cylinder length="0.02" radius="0.05"/>
-      </geometry>
-      <material name="blue"/>
-    </visual>
-    <collision>
-      <origin rpy="0 0 0" xyz="0 0 0"/>
-      <geometry>
-        <cylinder length="0.02" radius="0.05"/>
-      </geometry>
-    </collision-->
-    <inertial>
-      <origin rpy="0 0 0" xyz="0 0 0"/>
-      <mass value="${steer_front_mass}"/>
+    <xacro:solid_cylinder_inertial
+      xyz="0.0 0.0 0.0"
+      rpy="0.0 0.0 0.0"
+      mass="${steer_front_mass}"
+      radius="0.01"
+      length="0.01"/>
+    <!--inertial>
       <inertia ixx="0.0006583333333333334" ixy="0.0" ixz="0.0" iyy="0.0006583333333333334" iyz="0.0" izz="0.0012500000000000002"/>
-    </inertial>
+    </inertial-->
   </link>
   <joint name="front_left_steer_joint" type="revolute">
     <parent link="base_link"/>
     <child link="front_left_steer_link"/>
-    <origin rpy="0 0 ${pi}" xyz="${wheelbase} -0.048 0"/>
+    <origin rpy="0.0 0.0 ${pi}" xyz="${wheelbase} ${-steer_front_axe} 0.0"/>
     <axis xyz="0 0 1"/>
     <limit effort="10.0" lower="-0.7853981633974483" upper="0.7853981633974483" velocity="5.0"/>
@@ -232,26 +203,27 @@
   <link name="front_left_wheel_link">
     <visual>
-      <origin rpy="0 0 0" xyz="0 0 0"/>
-      <geometry>
-        <mesh filename="package://picar_description/meshes/WheelFrontLeft.dae" />
-      </geometry>
-      <material name="red"/>
-    </visual>
-    <collision>
-      <origin rpy="0 0 0" xyz="0 0 0"/>
-      <geometry>
-        <mesh filename="package://picar_description/meshes/WheelFrontLeft.dae" />
-      </geometry>
-    </collision>
-    <inertial>
-      <origin rpy="0 0 0" xyz="0 0 0"/>
-      <mass value="${wheel_front_mass}"/>
-      <inertia ixx="${wheel_front_mass*(3.0*wheel_front_radius*wheel_front_radius + wheel_front_width*wheel_front_width)/12.0}" ixy="0" ixz="0" iyy="${wheel_front_mass*(3.0*wheel_front_radius*wheel_front_radius + wheel_front_width*wheel_front_width)/12.0}" iyz="0" izz="${wheel_front_mass*wheel_front_radius*wheel_front_radius/2.0}"/>
-    </inertial>
+      <origin rpy="0.0 0.0 0.0" xyz="0.0 0.0 0.0"/>
+      <geometry>
+        <mesh filename="package://picar_description/meshes/WheelFrontRight.dae" />
+      </geometry>
+      <!--material name="red"/-->
+    </visual>
+    <collision>
+      <origin rpy="0.0 0.0 0.0" xyz="0.0 0.0 0.0"/>
+      <geometry>
+        <mesh filename="package://picar_description/meshes/WheelFrontRight.dae" />
+      </geometry>
+    </collision>
+    <xacro:solid_cylinder_inertial
+      xyz="0.0 0.0 0.0"
+      rpy="0.0 0.0 0.0"
+      mass="${wheel_front_mass}"
+      radius="${wheel_front_radius}"
+      length="${wheel_front_width}"/>
   </link>
   <joint name="front_left_wheel_joint" type="continuous">
     <parent link="front_left_steer_link"/>
     <child link="front_left_wheel_link"/>
-    <origin rpy="${-pi/2} 0 0" xyz="0 ${wheel_front_width/2} 0"/>
+    <origin rpy="${-pi/2} 0.0 0.0" xyz="0.0 ${wheel_front_width/2} 0.0"/>
     <axis xyz="0 0 -1"/>
   </joint>
@@ -288,26 +260,27 @@
   <link name="rear_right_wheel_link">
     <visual>
-      <origin rpy="0 0 0" xyz="0 0 0"/>
+      <origin rpy="0.0 0.0 0.0" xyz="0.0 0.0 0.0"/>
       <geometry>
         <mesh filename="package://picar_description/meshes/WheelRearRight.dae" />
       </geometry>
-      <material name="red"/>
-    </visual>
-    <collision>
-      <origin rpy="0 0 0" xyz="0 0 0"/>
+      <!--material name="red"/-->
+    </visual>
+    <collision>
+      <origin rpy="0.0 0.0 0.0" xyz="0.0 0.0 0.0"/>
       <geometry>
         <mesh filename="package://picar_description/meshes/WheelRearRight.dae" />
       </geometry>
     </collision>
-    <inertial>
-      <origin rpy="0 0 0" xyz="0 0 0"/>
-      <mass value="${wheel_rear_mass}"/>
-      <inertia ixx="${wheel_rear_mass*(3.0*wheel_rear_radius*wheel_rear_radius + wheel_rear_width*wheel_rear_width)/12.0}" ixy="0" ixz="0" iyy="${wheel_rear_mass*(3.0*wheel_rear_radius*wheel_rear_radius + wheel_rear_width*wheel_rear_width)/12.0}" iyz="0" izz="${wheel_rear_mass*wheel_rear_radius*wheel_rear_radius/2.0}"/>
-    </inertial>
+    <xacro:solid_cylinder_inertial
+      xyz="0.0 0.0 0.0"
+      rpy="0.0 0.0 0.0"
+      mass="${wheel_rear_mass}"
+      radius="${wheel_rear_radius}"
+      length="${wheel_rear_width}"/>
   </link>
   <joint name="rear_right_wheel_joint" type="continuous">
     <parent link="base_link"/>
     <child link="rear_right_wheel_link"/>
-    <origin rpy="${-pi/2} 0 0" xyz="0 0.055 0"/>
+    <origin rpy="${-pi/2} 0.0 0.0" xyz="0.0 ${steer_rear_axe} 0.0"/>
     <axis xyz="0 0 1"/>
   </joint>
@@ -329,26 +302,27 @@
   <link name="rear_left_wheel_link">
     <visual>
-      <origin rpy="0 0 0" xyz="0 0 0"/>
+      <origin rpy="0.0 0.0 0.0" xyz="0.0 0.0 0.0"/>
       <geometry>
         <mesh filename="package://picar_description/meshes/WheelRearLeft.dae" />
       </geometry>
-      <material name="red"/>
-    </visual>
-    <collision>
-      <origin rpy="0 0 0" xyz="0 0 0"/>
+      <!--material name="red"/-->
+    </visual>
+    <collision>
+      <origin rpy="0.0 0.0 0.0" xyz="0.0 0.0 0.0"/>
       <geometry>
         <mesh filename="package://picar_description/meshes/WheelRearLeft.dae" />
       </geometry>
     </collision>
-    <inertial>
-      <origin rpy="0 0 0" xyz="0 0 0"/>
-      <mass value="${wheel_rear_mass}"/>
-      <inertia ixx="${wheel_rear_mass*(3.0*wheel_rear_radius*wheel_rear_radius + wheel_rear_width*wheel_rear_width)/12.0}" ixy="0" ixz="0" iyy="${wheel_rear_mass*(3.0*wheel_rear_radius*wheel_rear_radius + wheel_rear_width*wheel_rear_width)/12.0}" iyz="0" izz="${wheel_rear_mass*wheel_rear_radius*wheel_rear_radius/2.0}"/>
-    </inertial>
+    <xacro:solid_cylinder_inertial
+      xyz="0.0 0.0 0.0"
+      rpy="0.0 0.0 0.0"
+      mass="${wheel_rear_mass}"
+      radius="${wheel_rear_radius}"
+      length="${wheel_rear_width}"/>
   </link>
   <joint name="rear_left_wheel_joint" type="continuous">
     <parent link="base_link"/>
     <child link="rear_left_wheel_link"/>
-    <origin rpy="${-pi/2} 0 0" xyz="0 -0.055 0"/>
+    <origin rpy="${-pi/2} 0.0 0.0" xyz="0.0 ${-steer_rear_axe} 0.0"/>
     <axis xyz="0 0 1"/>
   </joint>

Commit message: Update URDF model
Signed-off-by: Mickael Gaillard <mick.gaillard@gmail.com>

File: picar_description/urdf/config.xacro (robot description, xacro)
@@ -6,5 +6,6 @@
   <xacro:arg name="body_height"   default="0.029"/>
   <xacro:arg name="body_offset"   default="0.070"/>
-  <xacro:arg name="wheelbase"     default="0.140"/>
+  <xacro:arg name="wheelbase_h"     default="0.096"/>
+  <xacro:arg name="wheelbase_w"     default="0.140"/>
   <!-- Rear wheel -->
   <xacro:arg name="steer_rear_axe"     default="0.055"/>
@@ -14,5 +15,5 @@
   <!-- Front wheel -->
   <xacro:arg name="steer_front_mass"    default="0.031"/>
-  <xacro:arg name="steer_front_axe"     default="0.048"/>
+  <xacro:arg name="steer_front_axe"     default="0.048"/><!-- ${wheelbase_h/2} -->
   <xacro:arg name="wheel_front_mass"    default="0.023"/>
   <xacro:arg name="wheel_front_width"   default="0.026"/>

File: picar_description/urdf/converter.urdf.xacro (robot description, xacro)
@@ -6,5 +6,6 @@
   <xacro:property name="body_height" value="$(arg body_height)"/>
   <xacro:property name="body_offset" value="$(arg body_offset)"/>
-  <xacro:property name="wheelbase" value="$(arg wheelbase)"/>
+  <xacro:property name="wheelbase_h" value="$(arg wheelbase_h)"/>
+  <xacro:property name="wheelbase_w" value="$(arg wheelbase_w)"/>
   <xacro:property name="steer_rear_axe" value="$(arg steer_rear_axe)"/>
   <xacro:property name="wheel_rear_mass" value="$(arg wheel_rear_mass)"/>

File: picar_description/urdf/inertials.xacro (robot description, xacro)
@@ -2,7 +2,10 @@
 <!--  xacro macros for inertials.
     Define xacro macros for math constants and inertials:
+    - solid sphere
     - solid cuboid
     - solid cylinder
+    - Thick-walled cylinder
     - null (a placeholder inertial for logical link elements)
+    base on https://en.wikipedia.org/wiki/List_of_moments_of_inertia
  -->
 <robot name="inertials" xmlns:xacro="http://wiki.ros.org/xacro">
@@ -11,4 +14,28 @@
     <xacro:property name="math_pi_over_2" value="1.5707963267948966" />
     <xacro:property name="math_pi_over_4" value="0.785398163397448" />
+    <!-- Inertial for solid sphere with dimensions x y z  -->
+    <xacro:macro name="solid_sphere_inertial" params="rpy xyz mass radius">
+        <inertial>
+            <origin rpy="${rpy}" xyz="${xyz}"/>
+            <mass value="${mass}" />
+            <inertia
+                ixx="${mass * (radius * radius) * (2/5)}" ixy="0.0" ixz="0.0"
+                iyy="${mass * (radius * radius) * (2/5)}" iyz="0.0"
+                izz="${mass * (radius * radius) * (2/5)}">
+            </inertia>
+        </inertial>
+    </xacro:macro>
+    <!-- Inertial for Hollow sphere with dimensions x y z  -->
+    <xacro:macro name="hollow_sphere_inertial" params="rpy xyz mass radius">
+        <inertial>
+            <origin rpy="${rpy}" xyz="${xyz}"/>
+            <mass value="${mass}" />
+            <inertia
+                ixx="${mass * (radius * radius) * (2/3)}" ixy="0.0" ixz="0.0"
+                iyy="${mass * (radius * radius) * (2/3)}" iyz="0.0"
+                izz="${mass * (radius * radius) * (2/3)}">
+            </inertia>
+        </inertial>
+    </xacro:macro>
     <!-- Inertial for solid cuboid with dimensions x y z  -->
     <xacro:macro name="solid_cuboid_inertial" params="rpy xyz mass x y z">
@@ -17,7 +44,7 @@
             <mass value="${mass}" />
             <inertia
-                ixx="${mass * (y * y + z * z) / 12.0}" ixy="0.0" ixz="0.0"
-                iyy="${mass * (x * x + z * z) / 12.0}" iyz="0.0"
-                izz="${mass * (x * x + y * y) / 12.0}">
+                ixx="${mass * ((y * y) + (z * z)) / 12.0}" ixy="0.0" ixz="0.0"
+                iyy="${mass * ((x * x) + (z * z)) / 12.0}" iyz="0.0"
+                izz="${mass * ((x * x) + (y * y)) / 12.0}">
             </inertia>
         </inertial>
@@ -29,7 +56,18 @@
             <mass value="${mass}" />
             <inertia
-                ixx="${mass * (3.0 * radius * radius + length * length) / 12.0}" ixy="0.0" ixz="0.0"
-                iyy="${mass * (3.0 * radius * radius + length * length) / 12.0}" iyz="0.0"
+                ixx="${mass * (3.0 * (radius * radius) + (length * length)) / 12.0}" ixy="0.0" ixz="0.0"
+                iyy="${mass * (3.0 * (radius * radius) + (length * length)) / 12.0}" iyz="0.0"
                 izz="${mass * (radius * radius) / 2.0}" />
+        </inertial>
+    </xacro:macro>
+    <!-- Inertial for Thick-walled cylinder with (inner/outer)-radius and length aligned to z-axis  -->
+    <xacro:macro name="thickwalled_cylinder_inertial" params="rpy xyz mass inner_radius outer_radius length">
+        <inertial>
+            <origin rpy="${rpy}" xyz="${xyz}"/>
+            <mass value="${mass}" />
+            <inertia
+                ixx="${mass * (3.0 * ((outer_radius * outer_radius)+(inner_radius * inner_radius)) + (length * length)) / 12.0}" ixy="0.0" ixz="0.0"
+                iyy="${mass * (3.0 * ((outer_radius * outer_radius)+(inner_radius * inner_radius)) + (length * length)) / 12.0}" iyz="0.0"
+                izz="${mass * ((outer_radius * outer_radius)+(inner_radius * inner_radius)) / 2.0}" />
         </inertial>
     </xacro:macro>
@@ -38,5 +76,5 @@
         <inertial>
             <mass value="0.001"/>
-            <inertia ixx="9.049479166666668e-06" ixy="0" ixz="0" iyy="9.049479166666668e-06" iyz="0" izz="9.765625000000002e-06"/>
+            <inertia ixx="1.666666666667e-08" ixy="0" ixz="0" iyy="1.666666666667e-08" iyz="0" izz="1.666666666667e-08"/>
         </inertial>
     </xacro:macro>

File: picar_description/urdf/picar.urdf.xacro (robot description, xacro)
@@ -35,5 +35,5 @@
     </collision>
     <xacro:solid_cuboid_inertial
-        xyz="0.0 0.0 ${body_height/2}"
+        xyz="0.07 0.0 ${-body_height/2}"
         rpy="0.0 0.0 0.0"
         mass="${body_mass}"
@@ -47,10 +47,11 @@
   <!-- End Baselink -->
   <link name="front_steer_link">
-    <xacro:solid_cylinder_inertial
-      xyz="0.0 0.0 0.0"
-      rpy="0.0 0.0 0.0"
-      mass="0.03125"
+    <xacro:null_inertial />
+    <!--xacro:solid_cylinder_inertial
+      xyz="0.0 0.0 0.0"
+      rpy="0.0 0.0 0.0"
+      mass="0.00125"
       radius="0.01"
-      length="0.01"/>
+      length="0.01"/-->
     <!--inertia ixx="0.0006583333333333334" ixy="0.0" ixz="0.0" iyy="0.0006583333333333334" iyz="0.0" izz="0.0012500000000000002"/-->
   </link>
@@ -124,5 +125,5 @@
     <parent link="base_link"/>
     <child link="front_right_steer_link"/>
-    <origin rpy="0.0 0.0 0.0" xyz="${wheelbase} ${steer_front_axe} 0.0"/>
+    <origin rpy="0.0 0.0 0.0" xyz="${wheelbase_w} ${steer_front_axe} 0.0"/>
     <axis xyz="0 0 1"/>
     <limit effort="10.0" lower="-0.7853981633974483" upper="0.7853981633974483" velocity="5.0"/>
@@ -134,5 +135,4 @@
         <mesh filename="package://picar_description/meshes/WheelFrontRight.dae" />
       </geometry>
-      <!--material name="red"/-->
     </visual>
     <collision>
@@ -197,5 +197,5 @@
     <parent link="base_link"/>
     <child link="front_left_steer_link"/>
-    <origin rpy="0.0 0.0 ${pi}" xyz="${wheelbase} ${-steer_front_axe} 0.0"/>
+    <origin rpy="0.0 0.0 ${pi}" xyz="${wheelbase_w} ${-steer_front_axe} 0.0"/>
     <axis xyz="0 0 1"/>
     <limit effort="10.0" lower="-0.7853981633974483" upper="0.7853981633974483" velocity="5.0"/>
@@ -207,5 +207,4 @@
         <mesh filename="package://picar_description/meshes/WheelFrontRight.dae" />
       </geometry>
-      <!--material name="red"/-->
     </visual>
     <collision>
@@ -264,5 +263,4 @@
         <mesh filename="package://picar_description/meshes/WheelRearRight.dae" />
       </geometry>
-      <!--material name="red"/-->
     </visual>
     <collision>
@@ -306,5 +304,4 @@
         <mesh filename="package://picar_description/meshes/WheelRearLeft.dae" />
       </geometry>
-      <!--material name="red"/-->
     </visual>
     <collision>
