Commit message: Add more gazebo sensor
Signed-off-by: Mickael Gaillard <mick.gaillard@gmail.com>

File: picar_description/urdf/config.xacro (robot description, xacro)
@@ -1,4 +1,4 @@
 <?xml version="1.0" ?>
-<robot name="robot" xmlns:xacro="http://ros.org/wiki/xacro">
+<robot name="config" xmlns:xacro="http://ros.org/wiki/xacro">
   <xacro:arg name="body_mass"     default="1.000"/>
   <xacro:arg name="body_width"    default="0.078"/>

File: picar_description/urdf/converter.urdf.xacro (robot description, xacro)
@@ -1,4 +1,4 @@
 <?xml version="1.0" ?>
-<robot name="picar" xmlns:xacro="http://www.ros.org/wiki/xacro">
+<robot name="converter" xmlns:xacro="http://www.ros.org/wiki/xacro">
   <xacro:property name="body_mass" value="$(arg body_mass)"/>
   <xacro:property name="body_width" value="$(arg body_width)"/>

File: picar_description/urdf/materials.xacro (robot description, xacro)
@@ -1,4 +1,4 @@
 <?xml version="1.0" ?>
-<robot name="robot" xmlns:xacro="http://www.ros.org/wiki/xacro" >
+<robot name="materials" xmlns:xacro="http://www.ros.org/wiki/xacro" >
   <!-- Start Materials -->
   <material name="metal">

File: picar_description/urdf/picar.urdf.xacro (robot description, xacro)
@@ -9,4 +9,7 @@
   <xacro:include filename="$(find picar_description)/urdf/materials.xacro" />
   <xacro:include filename="$(find picar_description)/urdf/inertials.xacro" />
+  <xacro:include filename="$(find picar_description)/urdf/lidar.urdf.xacro" />
+  <xacro:include filename="$(find picar_description)/urdf/openni.urdf.xacro" />
+  <xacro:include filename="$(find picar_description)/urdf/imu.urdf.xacro" />
   <xacro:property name="robot_namespace" value="/picar"/>
   <!-- Gazebo plugins -->
@@ -20,4 +23,29 @@
     </plugin>
   </gazebo>
+  <!-- Start BaseFootprint -->
+  <!--link name="base_footprint">
+    <inertial>
+      <mass value="0.0001"/>
+      <origin xyz="0 0 0"/>
+      <inertia
+        ixx="0.0001" ixy="0.0" ixz="0.0"
+        iyy="0.0001" iyz="0.0"
+        izz="0.0001"/>
+    </inertial>
+    <visual>
+      <origin rpy="0 0 0" xyz="0 0 0"/>
+      <geometry>
+        <box size="0.001 0.001 0.001"/>
+      </geometry>
+    </visual>
+  </link>
+  <gazebo reference="base_footprint">
+    <turnGravityOff>false</turnGravityOff>
+  </gazebo>
+  <joint name="base_footprint_joint" type="fixed">
+    <origin rpy="0 0 0" xyz="0 0 0.04"/>
+    <parent link="base_footprint"/>
+    <child link="base_link"/>
+  </joint-->
   <!-- Start Baselink -->
   <link name="base_link">
@@ -59,5 +87,5 @@
     <parent link="base_link"/>
     <child link="front_steer_link"/>
-    <origin rpy="0.0 0.0 0.0" xyz="0.2 0 0.12000000000000001"/>
+    <origin rpy="0.0 0.0 0.0" xyz="${wheelbase_w} 0 0"/>
     <axis xyz="0 0 1"/>
     <limit effort="10.0" lower="${-pi}" upper="${pi}" velocity="5.0"/>
