Commit message: Fix Openni sensor for gazebo
Signed-off-by: Mickael Gaillard <mick.gaillard@gmail.com>

File: picar_description/urdf/lidar.urdf.xacro (robot description, xacro)
@@ -40,5 +40,5 @@
     <sensor type="ray" name="lidar">
       <pose>0 0 0 0 0 0</pose>
-      <visualize>true</visualize>
+      <visualize>false</visualize>
       <update_rate>5</update_rate>
       <ray>
@@ -64,5 +64,5 @@
       <plugin name="gazebo_ros_lidar" filename="libgazebo_ros_laser.so">
         <topicName>/picar/laser/scan</topicName>
-        <frameName>sensor_laser</frameName>
+        <frameName>/sensor_laser</frameName>
       </plugin>
     </sensor>

File: picar_description/urdf/openni.urdf.xacro (robot description, xacro)
@@ -1,71 +1,138 @@
 <?xml version="1.0" ?>
-<robot name="openni" xmlns:xacro="http://www.ros.org/wiki/xacro">
+<robot name="sensor_xtion_pro" xmlns:xacro="http://www.ros.org/wiki/xacro">
   <xacro:include filename="$(find picar_description)/urdf/inertials.xacro" />
-  <xacro:property name="camera_size_x" value="0.03"/>
-  <xacro:property name="camera_size_y" value="0.03"/>
-  <xacro:property name="camera_size_z" value="0.04"/>
-  <xacro:property name="camera_origin_x" value="0.065"/>
-  <xacro:property name="camera_origin_y" value="0"/>
-  <xacro:property name="camera_origin_z" value="0.035"/>
-  <xacro:property name="link_name" value="camera_link"/>
-  <xacro:property name="camera_name" value="camera0"/>
-  <xacro:property name="frame_name" value="camera_link"/>
-  <!-- Camera -->
-  <link name="${link_name}">
+  <!-- Xacro properties -->
+  <xacro:property name="camera_origin_x" value="0.19825"/>
+  <xacro:property name="camera_origin_y" value="0.0"/>
+  <xacro:property name="camera_origin_z" value="${0.113-(0.027+0.002)}"/>
+  <xacro:property name="asus_xtion_pro_depth_rel_rgb_py" value="0.0270" />
+  <xacro:property name="asus_xtion_pro_cam_rel_rgb_py"   value="-0.0220" />
+  <xacro:property name="M_SCALE" value="0.001"/>
+  <joint name="camera_rgb_joint" type="fixed">
+    <origin xyz="${camera_origin_x} ${camera_origin_y} ${camera_origin_z}"
+            rpy="0 0 0"/>
+    <parent link="base_link"/>
+    <child link="camera_rgb_frame" />
+  </joint>
+  <link name="camera_rgb_frame">
+    <inertial>
+      <mass value="0.001" />
+      <origin xyz="0 0 0" />
+      <inertia ixx="0.0001" ixy="0.0" ixz="0.0"
+        iyy="0.0001" iyz="0.0"
+        izz="0.0001" />
+    </inertial>
+  </link>
+  <joint name="camera_rgb_optical_joint" type="fixed">
+    <origin xyz="0 0 0" rpy="${-pi/2} 0 ${-pi/2}" />
+    <parent link="camera_rgb_frame" />
+    <child link="camera_rgb_optical_frame" />
+  </joint>
+  <link name="camera_rgb_optical_frame">
+    <inertial>
+      <mass value="0.001" />
+      <origin xyz="0 0 0" />
+      <inertia ixx="0.0001" ixy="0.0" ixz="0.0"
+        iyy="0.0001" iyz="0.0"
+        izz="0.0001" />
+    </inertial>
+  </link>
+  <joint name="camera_joint" type="fixed">
+    <origin xyz="0 ${asus_xtion_pro_cam_rel_rgb_py} 0"
+            rpy="0 0 0"/>
+    <parent link="camera_rgb_frame"/>
+    <child link="camera_link"/>
+  </joint>
+  <link name="camera_link">
     <visual>
-      <origin xyz="0 0 0" rpy="0 0 0"/>
+      <origin xyz="-0.01 0.0 0.0" rpy="${-pi/2} ${-pi} ${-pi/2}"/>
       <geometry>
-        <box size="${camera_size_x} ${camera_size_y} ${camera_size_z}"/>
+        <mesh filename="package://picar_description/meshes/sensors/asus_xtion_pro_live.dae" scale="${M_SCALE} ${M_SCALE} ${M_SCALE}"/>
       </geometry>
-      <material name="red"/>
     </visual>
     <collision>
-      <origin xyz="0 0 0" rpy="0 0 0"/>
+      <origin xyz="0.0 0.0 0.0" rpy="0 0 0" />
       <geometry>
-        <box size="${camera_size_x} ${camera_size_y} ${camera_size_z}"/>
-      </geometry>
+      <box size="0.0730 0.2760 0.0720"/>
+    </geometry>
     </collision>
-    <xacro:solid_cuboid_inertial
-        xyz="0.0 0.0 0.0"
-        rpy="0.0 0.0 0.0"
-        mass="0.2"
-        x="0.01"
-        y="0.01"
-        z="0.01" />
+    <inertial>
+      <mass value="0.170" />
+      <origin xyz="0 0 0" />
+      <inertia ixx="0.001152600" ixy="0.0" ixz="0.0"
+                iyy="0.000148934" iyz="0.0"
+                izz="0.001154654" />
+    </inertial>
   </link>
-  <joint name="camera_joint" type="fixed">
-    <axis xyz="0 1 0" />
-    <origin xyz="${camera_origin_x} ${camera_origin_y} ${camera_origin_z}" rpy="0 0 0"/>
-    <parent link="base_link"/>
-    <child link="${link_name}"/>
+  <joint name="camera_depth_joint" type="fixed">
+    <origin xyz="0 ${asus_xtion_pro_depth_rel_rgb_py} 0" rpy="0 0 0" />
+    <parent link="camera_rgb_frame" />
+    <child link="camera_depth_frame" />
   </joint>
-  <!-- camera -->
-  <gazebo reference="${link_name}">
-    <sensor name="${link_name}_camera" type="depth">
+  <link name="camera_depth_frame">
+    <inertial>
+      <mass value="0.01" />
+      <origin xyz="0 0 0" />
+      <inertia ixx="0.001" ixy="0.0" ixz="0.0"
+        iyy="0.001" iyz="0.0"
+        izz="0.001" />
+    </inertial>
+  </link>
+  <joint name="camera_depth_optical_joint" type="fixed">
+    <origin xyz="0 0 0" rpy="${-pi/2} 0 ${-pi/2}" />
+    <parent link="camera_depth_frame" />
+    <child link="camera_depth_optical_frame" />
+  </joint>
+  <link name="camera_depth_optical_frame">
+    <inertial>
+      <mass value="0.001" />
+      <origin xyz="0 0 0" />
+      <inertia ixx="0.0001" ixy="0.0" ixz="0.0"
+        iyy="0.0001" iyz="0.0"
+        izz="0.0001" />
+    </inertial>
+  </link>
+  <!-- generate an optical frame
+  http://www.ros.org/reps/rep-0103.html#suffix-frames
+  so that ros and opencv can operate on the camera frame correctly
+  -->
+  <joint name="camera_optical_joint" type="fixed">
+    <!-- these values have to be these values otherwise the gazebo camera
+        image won't be aligned properly with the frame it is supposedly
+        originating from -->
+    <origin xyz="0 0 0" rpy="${-pi/2} 0 ${-pi/2}"/>
+    <parent link="camera_link"/>
+    <child link="camera_link_optical"/>
+  </joint>
+  <link name="camera_link_optical" />
+    <!-- RGBD sensor for simulation, same as Kinect -->
+  <gazebo reference="camera_link">
+    <sensor name="camera" type="depth">
+      <always_on>true</always_on>
       <update_rate>20</update_rate>
       <camera>
-        <horizontal_fov>1.047198</horizontal_fov>
+        <horizontal_fov>${60.0*pi/180.0}</horizontal_fov>
         <image>
           <width>640</width>
           <height>480</height>
-          <format>R8G8B8</format>
+          <format>B8G8R8</format>
         </image>
         <clip>
           <near>0.05</near>
-          <far>3</far>
+          <far>8.0</far>
         </clip>
       </camera>
-      <plugin name="${link_name}_controller" filename="libgazebo_ros_openni_kinect.so">
-        <baseline>0.2</baseline>
+      <plugin name="camera_controller" filename="libgazebo_ros_openni_kinect.so">
+        <baseline>0.1</baseline>
         <alwaysOn>true</alwaysOn>
-        <updateRate>1.0</updateRate>
-        <cameraName>${camera_name}_ir</cameraName>
-        <imageTopicName>color/image_raw</imageTopicName>
-        <cameraInfoTopicName>color/camera_info</cameraInfoTopicName>
+        <updateRate>10.0</updateRate>
+        <cameraName>camera_ir</cameraName>
+        <imageTopicName>rgb/image_raw</imageTopicName>
+        <cameraInfoTopicName>rgb/camera_info</cameraInfoTopicName>
         <depthImageTopicName>depth/image_raw</depthImageTopicName>
         <depthImageInfoTopicName>depth/camera_info</depthImageInfoTopicName>
         <pointCloudTopicName>depth/points</pointCloudTopicName>
-        <frameName>${frame_name}</frameName>
-        <pointCloudCutoff>0.5</pointCloudCutoff>
+        <frameName>/camera_link_optical</frameName><!--camera_depth_optical_frame-->
+        <pointCloudCutoff>0.4</pointCloudCutoff>
         <pointCloudCutoffMax>3.0</pointCloudCutoffMax>
         <distortionK1>0.00000001</distortionK1>
@@ -82,39 +149,3 @@
     </sensor>
   </gazebo>
-  <!--gazebo reference="camera_link">
-    <sensor type="camera" name="camera0">
-      <update_rate>30.0</update_rate>
-      <camera name="head">
-        <horizontal_fov>1.3962634</horizontal_fov>
-        <image>
-          <width>800</width>
-          <height>800</height>
-          <format>R8G8B8</format>
-        </image>
-        <clip>
-          <near>0.02</near>
-          <far>300</far>
-        </clip>
-        <noise>
-          <type>gaussian</type>
-          <mean>0.0</mean>
-          <stddev>0.007</stddev>
-        </noise>
-      </camera>
-      <plugin name="camera_controller" filename="libgazebo_ros_camera.so">
-        <alwaysOn>true</alwaysOn>
-        <updateRate>0.0</updateRate>
-        <cameraName>camera0</cameraName>
-        <imageTopicName>image_raw</imageTopicName>
-        <cameraInfoTopicName>camera_info</cameraInfoTopicName>
-        <frameName>camera_link</frameName>
-        <hackBaseline>0.07</hackBaseline>
-        <distortionK1>0.0</distortionK1>
-        <distortionK2>0.0</distortionK2>
-        <distortionK3>0.0</distortionK3>
-        <distortionT1>0.0</distortionT1>
-        <distortionT2>0.0</distortionT2>
-      </plugin>
-    </sensor>
-  </gazebo-->
 </robot>

File: picar_description/urdf/picar.urdf.xacro (robot description, xacro)
@@ -24,13 +24,5 @@
   </gazebo>
   <!-- Start BaseFootprint -->
-  <!--link name="base_footprint">
-    <inertial>
-      <mass value="0.0001"/>
-      <origin xyz="0 0 0"/>
-      <inertia
-        ixx="0.0001" ixy="0.0" ixz="0.0"
-        iyy="0.0001" iyz="0.0"
-        izz="0.0001"/>
-    </inertial>
+  <link name="base_footprint">
     <visual>
       <origin rpy="0 0 0" xyz="0 0 0"/>
@@ -40,12 +32,9 @@
     </visual>
   </link>
-  <gazebo reference="base_footprint">
-    <turnGravityOff>false</turnGravityOff>
-  </gazebo>
   <joint name="base_footprint_joint" type="fixed">
     <origin rpy="0 0 0" xyz="0 0 0.04"/>
     <parent link="base_footprint"/>
     <child link="base_link"/>
-  </joint-->
+  </joint>
   <!-- Start Baselink -->
   <link name="base_link">

Commit message: Add new Teleop joy (FS-i6x)
Signed-off-by: Mickael Gaillard <mick.gaillard@gmail.com>

File: picar_description/urdf/lidar.urdf.xacro (robot description, xacro)
@@ -2,10 +2,9 @@
 <robot name="lidar" xmlns:xacro="http://www.ros.org/wiki/xacro">
   <xacro:include filename="$(find picar_description)/urdf/inertials.xacro" />
-  <xacro:property name="laser_size_x" value="0.03"/>
-  <xacro:property name="laser_size_y" value="0.03"/>
-  <xacro:property name="laser_size_z" value="0.04"/>
-  <xacro:property name="laser_origin_x" value="0.065"/>
-  <xacro:property name="laser_origin_y" value="0"/>
-  <xacro:property name="laser_origin_z" value="0.035"/>
+  <xacro:property name="laser_size_radius" value="0.038"/>
+  <xacro:property name="laser_size_length" value="0.025"/>
+  <xacro:property name="laser_origin_x" value="0.0"/>
+  <xacro:property name="laser_origin_y" value="0.0"/>
+  <xacro:property name="laser_origin_z" value="0.120"/>
   <!-- LIDAR -->
   <link name="sensor_laser">
@@ -13,21 +12,20 @@
       <origin xyz="0 0 0" rpy="0 0 0"/>
       <geometry>
-        <box size="${laser_size_x} ${laser_size_y} ${laser_size_z}"/>
+        <cylinder length="${laser_size_length}" radius="${laser_size_radius}"/>
       </geometry>
-      <material name="blue"/>
+      <material name="black"/>
     </visual>
     <collision>
       <origin xyz="0 0 0" rpy="0 0 0"/>
       <geometry>
-        <box size="${laser_size_x} ${laser_size_y} ${laser_size_z}"/>
+        <cylinder length="${laser_size_length}" radius="${laser_size_radius}"/>
       </geometry>
     </collision>
-    <xacro:solid_cuboid_inertial
+    <xacro:solid_cylinder_inertial
         xyz="0.0 0.0 0.0"
         rpy="0.0 0.0 0.0"
         mass="0.2"
-        x="${laser_size_x}"
-        y="${laser_size_y}"
-        z="${laser_size_z}" />
+        length="${laser_size_length}"
+        radius="${laser_size_radius}"/>
   </link>
   <joint name="sensor_laser_joint" type="fixed">
@@ -38,4 +36,5 @@
   <!--Gazebo Laser Plugin-->
   <gazebo reference="sensor_laser">
+    <material>Gazebo/Black</material>
     <sensor type="ray" name="lidar">
       <pose>0 0 0 0 0 0</pose>
@@ -45,5 +44,5 @@
         <scan>
           <horizontal>
-            <samples>8000</samples>
+            <samples>500</samples>
             <resolution>1</resolution>
             <min_angle>-3.14159265359</min_angle>
@@ -52,7 +51,7 @@
         </scan>
         <range>
-          <min>0.10</min>
-          <max>30.0</max>
-          <resolution>0.01</resolution>
+          <min>0.15</min>
+          <max>12.0</max>
+          <resolution>0.5</resolution>
         </range>
         <noise>
@@ -63,5 +62,5 @@
       </ray>
       <plugin name="gazebo_ros_lidar" filename="libgazebo_ros_laser.so">
-        <topicName>/picar/laser/scan</topicName>
+        <topicName>laser/scan</topicName>
         <frameName>/sensor_laser</frameName>
       </plugin>

File: picar_description/urdf/openni.urdf.xacro (robot description, xacro)
@@ -52,8 +52,8 @@
     </visual>
     <collision>
-      <origin xyz="0.0 0.0 0.0" rpy="0 0 0" />
+      <origin xyz="-0.01 0.0 0.0" rpy="${-pi/2} ${-pi} ${-pi/2}"/>
       <geometry>
-      <box size="0.0730 0.2760 0.0720"/>
-    </geometry>
+        <mesh filename="package://picar_description/meshes/sensors/asus_xtion_pro_live.dae" scale="${M_SCALE} ${M_SCALE} ${M_SCALE}"/>
+      </geometry>
     </collision>
     <inertial>

Commit message: Add many update for navigation
Signed-off-by: Mickael Gaillard <mick.gaillard@gmail.com>

File: picar_description/urdf/lidar.urdf.xacro (robot description, xacro)
@@ -40,9 +40,9 @@
       <pose>0 0 0 0 0 0</pose>
       <visualize>false</visualize>
-      <update_rate>5</update_rate>
+      <update_rate>10</update_rate>
       <ray>
         <scan>
           <horizontal>
-            <samples>500</samples>
+            <samples>8000</samples>
             <resolution>1</resolution>
             <min_angle>-3.14159265359</min_angle>

File: picar_description/urdf/openni.urdf.xacro (robot description, xacro)
@@ -16,11 +16,11 @@
   </joint>
   <link name="camera_rgb_frame">
-    <inertial>
+    <!--inertial>
       <mass value="0.001" />
-      <origin xyz="0 0 0" />
-      <inertia ixx="0.0001" ixy="0.0" ixz="0.0"
-        iyy="0.0001" iyz="0.0"
-        izz="0.0001" />
-    </inertial>
+      <origin xyz="0 0 0" rpy="0 0 0" />
+      <inertia  ixx="0.0001" ixy="0.0" ixz="0.0"
+                iyy="0.0001" iyz="0.0"
+                izz="0.0001" />
+    </inertial-->
   </link>
   <joint name="camera_rgb_optical_joint" type="fixed">
@@ -30,11 +30,11 @@
   </joint>
   <link name="camera_rgb_optical_frame">
-    <inertial>
+    <!--inertial>
       <mass value="0.001" />
-      <origin xyz="0 0 0" />
-      <inertia ixx="0.0001" ixy="0.0" ixz="0.0"
-        iyy="0.0001" iyz="0.0"
-        izz="0.0001" />
-    </inertial>
+      <origin xyz="0 0 0" rpy="0 0 0" />
+      <inertia  ixx="0.0001" ixy="0.0" ixz="0.0"
+                iyy="0.0001" iyz="0.0"
+                izz="0.0001" />
+    </inertial-->
   </link>
   <joint name="camera_joint" type="fixed">
@@ -57,11 +57,18 @@
       </geometry>
     </collision>
-    <inertial>
+    <xacro:solid_cuboid_inertial
+        xyz="0.0 0.0 0.0"
+        rpy="${-pi/2} ${-pi} ${-pi/2}"
+        mass="0.170"
+        x="0.18"
+        y="0.035"
+        z="0.025" />
+    <!--inertial>
       <mass value="0.170" />
-      <origin xyz="0 0 0" />
-      <inertia ixx="0.001152600" ixy="0.0" ixz="0.0"
+      <origin xyz="0 0 0" rpy="0 0 0" />
+      <inertia  ixx="0.001152600" ixy="0.0" ixz="0.0"
                 iyy="0.000148934" iyz="0.0"
                 izz="0.001154654" />
-    </inertial>
+    </inertial-->
   </link>
   <joint name="camera_depth_joint" type="fixed">
@@ -71,11 +78,11 @@
   </joint>
   <link name="camera_depth_frame">
-    <inertial>
+    <!--inertial>
       <mass value="0.01" />
-      <origin xyz="0 0 0" />
-      <inertia ixx="0.001" ixy="0.0" ixz="0.0"
-        iyy="0.001" iyz="0.0"
-        izz="0.001" />
-    </inertial>
+      <origin xyz="0 0 0" rpy="0 0 0" />
+      <inertia  ixx="0.001" ixy="0.0" ixz="0.0"
+                iyy="0.001" iyz="0.0"
+                izz="0.001" />
+    </inertial-->
   </link>
   <joint name="camera_depth_optical_joint" type="fixed">
@@ -85,11 +92,11 @@
   </joint>
   <link name="camera_depth_optical_frame">
-    <inertial>
+    <!--inertial>
       <mass value="0.001" />
-      <origin xyz="0 0 0" />
-      <inertia ixx="0.0001" ixy="0.0" ixz="0.0"
-        iyy="0.0001" iyz="0.0"
-        izz="0.0001" />
-    </inertial>
+      <origin xyz="0 0 0" rpy="0 0 0" />
+      <inertia  ixx="0.0001" ixy="0.0" ixz="0.0"
+                iyy="0.0001" iyz="0.0"
+                izz="0.0001" />
+    </inertial-->
   </link>
   <!-- generate an optical frame

File: picar_description/urdf/picar.urdf.xacro (robot description, xacro)
@@ -11,5 +11,5 @@
   <xacro:include filename="$(find picar_description)/urdf/lidar.urdf.xacro" />
   <xacro:include filename="$(find picar_description)/urdf/openni.urdf.xacro" />
-  <xacro:include filename="$(find picar_description)/urdf/imu.urdf.xacro" />
+  <!--xacro:include filename="$(find picar_description)/urdf/imu.urdf.xacro" /-->
   <xacro:property name="robot_namespace" value="/picar"/>
   <!-- Gazebo plugins -->
@@ -52,5 +52,5 @@
     </collision>
     <xacro:solid_cuboid_inertial
-        xyz="0.07 0.0 ${-body_height/2}"
+        xyz="0.07 0.0 0.0"
         rpy="0.0 0.0 0.0"
         mass="${body_mass}"
